File: flowerbed/hw/Flowerbed.kicad_sch (KiCad schematic)
At the start: 24 parts, among them J2 Conn_01x04, U2 STM32G030F6Px, U2 VL53L0X, U3 W25Q16JVSS, U4 MAX98357AETE+, X1 12.288MHz

Commit message: Flowerbed unit layout?
Connections:
- net ACT_LED: now also R3.1; no longer D1.2 (A)
- net GND: now also D1.1 (K); no longer R3.2
- new net: D1.2 (A), R3.2
Changed lines of the file:
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@@
+    )
+  )
+  (symbol (lib_id "Device:R") (at 78.105 85.725 90) (unit 1)
+    (in_bom yes) (on_board yes) (dnp no)
+    (property "Reference" "R3" (at 78.105 80.01 90)
+      (effects (font (size 1.27 1.27)))
+    )
+    (property "Value" "2k TBD" (at 78.105 82.55 90)
+      (effects (font (size 1.27 1.27)))
+    )
+    (property "Footprint" "Resistor_SMD:R_0603_1608Metric" (at 78.105 87.503 90)
+      (effects (font (size 1.27 1.27)) hide)
+    )
+    (property "Datasheet" "~" (at 78.105 85.725 0)
+      (effects (font (size 1.27 1.27)) hide)
+    )
+    (pin "2")
+    (pin "1")
+    (instances
+      (project "Flowerbed"
+        (path "/ee02efde-3d2c-44cf-8dc7-72cfd16bb7ed"
+          (reference "R3") (unit 1)
+        )
+      )
     )
   )
@@
     )
   )
+  (symbol (lib_id "Device:LED") (at 88.265 85.725 180) (unit 1)
+    (in_bom yes) (on_board yes) (dnp no)
+    (property "Reference" "D1" (at 88.9 79.375 0)
+      (effects (font (size 1.27 1.27)))
+    )
+    (property "Value" "Green" (at 88.9 81.915 0)
+      (effects (font (size 1.27 1.27)))
+    )
+    (property "Footprint" "LED_SMD:LED_0603_1608Metric" (at 88.265 85.725 0)
+      (effects (font (size 1.27 1.27)) hide)
+    )
+    (property "Datasheet" "~" (at 88.265 85.725 0)
+      (effects (font (size 1.27 1.27)) hide)
+    )
+    (pin "2")
+    (pin "1")
+    (instances
+      (project "Flowerbed"
+        (path "/ee02efde-3d2c-44cf-8dc7-72cfd16bb7ed"
+          (reference "D1") (unit 1)
+        )
+      )
+    )
+  )
   (symbol (lib_id "Connector_Generic:Conn_01x04") (at 30.48 45.72 0) (mirror y) (unit 1)
     (in_bom yes) (on_board yes) (dnp no)
@@
     )
   )
-  (symbol (lib_id "Device:R") (at 88.265 85.725 90) (unit 1)
-    (in_bom yes) (on_board yes) (dnp no)
-    (property "Reference" "R3" (at 88.265 80.01 90)
-      (effects (font (size 1.27 1.27)))
-    )
-    (property "Value" "2k TBD" (at 88.265 82.55 90)
-      (effects (font (size 1.27 1.27)))
-    )
-    (property "Footprint" "Resistor_SMD:R_0603_1608Metric" (at 88.265 87.503 90)
-      (effects (font (size 1.27 1.27)) hide)
-    )
-    (property "Datasheet" "~" (at 88.265 85.725 0)
-      (effects (font (size 1.27 1.27)) hide)
-    )
-    (pin "2")
-    (pin "1")
-    (instances
-      (project "Flowerbed"
-        (path "/ee02efde-3d2c-44cf-8dc7-72cfd16bb7ed"
-          (reference "R3") (unit 1)
-        )
-      )
-    )
-  )
   (symbol (lib_id "power:GND") (at 194.945 127 0) (unit 1)
     (in_bom yes) (on_board yes) (dnp no) (fields_autoplaced)
@@
         )
       )
-    )
-  )
-  (symbol (lib_id "Device:LED") (at 78.105 85.725 180) (unit 1)
-    (in_bom yes) (on_board yes) (dnp no)
-    (property "Reference" "D1" (at 78.74 79.375 0)
-      (effects (font (size 1.27 1.27)))
-    )
-    (property "Value" "Green" (at 78.74 81.915 0)
-      (effects (font (size 1.27 1.27)))
-    )
-    (property "Footprint" "LED_SMD:LED_0603_1608Metric" (at 78.105 85.725 0)
-      (effects (font (size 1.27 1.27)) hide)
-    )
-    (property "Datasheet" "~" (at 78.105 85.725 0)
-      (effects (font (size 1.27 1.27)) hide)
-    )
-    (pin "2")
-    (pin "1")
-    (instances
-      (project "Flowerbed"
-        (path "/ee02efde-3d2c-44cf-8dc7-72cfd16bb7ed"
-          (reference "D1") (unit 1)
-        )
-      )

Commit message: (WIP) Add flowerbed central schematic
Parts:
- renumbered J2 to J1
Changed lines of the file:
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@@
   (junction (at 38.1 43.18) (diameter 0) (color 0 0 0 0)
   )
-  (junction (at 38.1 43.815) (diameter 0) (color 0 0 0 0)
-  )
   (junction (at 80.01 51.435) (diameter 0) (color 0 0 0 0)
   )
@@
   )
   (junction (at 67.31 48.26) (diameter 0) (color 0 0 0 0)
+  )
+  (junction (at 38.1 44.45) (diameter 0) (color 0 0 0 0)
   )
   (junction (at 135.255 40.005) (diameter 0) (color 0 0 0 0)
@@
     (stroke (width 0) (type default))
   )
-  (wire (pts (xy 43.815 43.815) (xy 38.1 43.815))
-    (stroke (width 0) (type default))
-  )
   (wire (pts (xy 92.075 85.725) (xy 94.615 85.725))
     (stroke (width 0) (type default))
@@
     (stroke (width 0) (type default))
   )
-  (wire (pts (xy 43.815 45.72) (xy 43.815 43.815))
-    (stroke (width 0) (type default))
-  )
-  (wire (pts (xy 35.56 43.815) (xy 38.1 43.815))
+  (wire (pts (xy 43.815 45.72) (xy 43.815 44.45))
+    (stroke (width 0) (type default))
+  )
+  (wire (pts (xy 35.56 44.45) (xy 38.1 44.45))
     (stroke (width 0) (type default))
   )
@@
     (stroke (width 0) (type default))
   )
+  (wire (pts (xy 38.1 44.45) (xy 43.815 44.45))
+    (stroke (width 0) (type default))
+  )
   (wire (pts (xy 187.325 74.295) (xy 179.705 74.295))
     (stroke (width 0) (type default))
@@
     (stroke (width 0) (type default))
   )
-  (wire (pts (xy 35.56 45.72) (xy 35.56 43.815))
+  (wire (pts (xy 35.56 45.72) (xy 35.56 44.45))
     (stroke (width 0) (type default))
   )
@@
       (project "Flowerbed"
         (path "/ee02efde-3d2c-44cf-8dc7-72cfd16bb7ed"
-          (reference "J1") (unit 1)
+          (reference "J2") (unit 1)
         )
       )
@@
   (symbol (lib_id "Connector_Generic:Conn_01x04") (at 30.48 45.72 0) (mirror y) (unit 1)
     (in_bom yes) (on_board yes) (dnp no)
-    (property "Reference" "J2" (at 26.67 46.99 0)
+    (property "Reference" "J1" (at 26.67 46.99 0)
       (effects (font (size 1.27 1.27)))
     )
@@
       (project "Flowerbed"
         (path "/ee02efde-3d2c-44cf-8dc7-72cfd16bb7ed"
-          (reference "J2") (unit 1)
+          (reference "J1") (unit 1)
         )
       )
@@
     )
   )
-  (symbol (lib_id "power:VDD") (at 38.1 43.18 0) (unit 1)
-    (in_bom yes) (on_board yes) (dnp no) (fields_autoplaced)
-    (property "Reference" "#PWR014" (at 38.1 46.99 0)
-      (effects (font (size 1.27 1.27)) hide)
-    )
-    (property "Value" "VDD" (at 38.1 38.735 0)
-      (effects (font (size 1.27 1.27)))
-    )
-    (property "Footprint" "" (at 38.1 43.18 0)
-      (effects (font (size 1.27 1.27)) hide)
-    )
-    (property "Datasheet" "" (at 38.1 43.18 0)
+  (symbol (lib_id "power:VDD") (at 38.1 42.545 0) (unit 1)
+    (in_bom yes) (on_board yes) (dnp no) (fields_autoplaced)
+    (property "Reference" "#PWR014" (at 38.1 46.355 0)
+      (effects (font (size 1.27 1.27)) hide)
+    )
+    (property "Value" "VDD" (at 38.1 38.1 0)
+      (effects (font (size 1.27 1.27)))
+    )
+    (property "Footprint" "" (at 38.1 42.545 0)
+      (effects (font (size 1.27 1.27)) hide)
+    )
+    (property "Datasheet" "" (at 38.1 42.545 0)
       (effects (font (size 1.27 1.27)) hide)
     )
@@
     )
   )
-  (symbol (lib_id "power:GND") (at 38.1 43.815 0) (unit 1)
-    (in_bom yes) (on_board yes) (dnp no) (fields_autoplaced)
-    (property "Reference" "#PWR023" (at 38.1 50.165 0)
-      (effects (font (size 1.27 1.27)) hide)
-    )
-    (property "Value" "GND" (at 38.1 48.26 0)
-      (effects (font (size 1.27 1.27)) hide)
-    )
-    (property "Footprint" "" (at 38.1 43.815 0)
-      (effects (font (size 1.27 1.27)) hide)
-    )
-    (property "Datasheet" "" (at 38.1 43.815 0)
-      (effects (font (size 1.27 1.27)) hide)
-    )
+  (symbol (lib_id "power:GND") (at 38.1 44.45 0) (unit 1)
+    (in_bom yes) (on_board yes) (dnp no) (fields_autoplaced)
+    (property "Reference" "#PWR023" (at 38.1 50.8 0)
+      (effects (font (size 1.27 1.27)) hide)
+    )
+    (property "Value" "GND" (at 38.1 48.895 0)
+      (effects (font (size 1.27 1.27)) hide)
+    )
+    (property "Footprint" "" (at 38.1 44.45 0)
+      (effects (font (size 1.27 1.27)) hide)
+    )
+    (property "Datasheet" "" (at 38.1 44.45 0)
+      (effects (font (size 1.27 1.27)) hide)
+    )

Commit message: Route flowerbed unit (!)
Parts:
- C2, C3: footprint Capacitor_SMD:C_0603_1608Metric -> Capacitor_SMD:C_0402_1005Metric
- U4: footprint Package_DFN_QFN:QFN-16-1EP_3x3mm_P0.5mm_EP1.45x1.45mm -> Flowerbed_footprints:QFN-16_3x3mm_P0.5mm
Connections:
- net SPI2_CSx: now also U2.9 (PA2); no longer U2.8 (PA1)
Changed lines of the file:
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@@
   (junction (at 147.32 47.625) (diameter 0) (color 0 0 0 0)
   )
-  (no_connect (at 149.225 59.055))
   (no_connect (at 238.125 123.19))
   (no_connect (at 108.585 53.975))
@@
   (no_connect (at 246.38 35.56))
   (no_connect (at 149.225 69.215))
+  (no_connect (at 149.225 56.515))
   (no_connect (at 191.135 125.73))
   (no_connect (at 212.725 148.59))
@@
     (effects (font (size 1.27 1.27) italic) (justify left bottom))
   )
-  (text "GPIO" (at 163.195 57.785 0)
-    (effects (font (size 1.27 1.27) italic) (justify left bottom))
-  )
   (text "PA3 AF0" (at 163.195 62.865 0)
     (effects (font (size 1.27 1.27) italic) (justify left bottom))
@@
   )
   (text "PA0 AF0" (at 163.195 55.245 0)
+    (effects (font (size 1.27 1.27) italic) (justify left bottom))
+  )
+  (text "GPIO" (at 163.195 60.325 0)
     (effects (font (size 1.27 1.27) italic) (justify left bottom))
   )
@@
     )
   )
+  (global_label "SPI2_CSx" (shape bidirectional) (at 149.225 59.055 0) (fields_autoplaced)
+    (effects (font (size 1.27 1.27)) (justify left))
+    (property "Intersheetrefs" "${INTERSHEET_REFS}" (at 162.0905 59.055 0)
+      (effects (font (size 1.27 1.27)) (justify left) hide)
+    )
+  )
   (global_label "SPI2_MISO" (shape bidirectional) (at 229.235 78.105 180) (fields_autoplaced)
     (effects (font (size 1.27 1.27)) (justify right))
@@
     )
   )
-  (global_label "SPI2_CSx" (shape bidirectional) (at 149.225 56.515 0) (fields_autoplaced)
-    (effects (font (size 1.27 1.27)) (justify left))
-    (property "Intersheetrefs" "${INTERSHEET_REFS}" (at 162.0905 56.515 0)
-      (effects (font (size 1.27 1.27)) (justify left) hide)
-    )
-  )
   (global_label "I2S1_CK" (shape bidirectional) (at 149.225 66.675 0) (fields_autoplaced)
     (effects (font (size 1.27 1.27)) (justify left))
@@
       (effects (font (size 1.27 1.27)))
     )
-    (property "Footprint" "Package_DFN_QFN:QFN-16-1EP_3x3mm_P0.5mm_EP1.45x1.45mm" (at 234.315 110.49 0)
+    (property "Footprint" "Flowerbed_footprints:QFN-16_3x3mm_P0.5mm" (at 234.315 110.49 0)
       (effects (font (size 1.27 1.27)) (justify left) hide)
     )
@@
       (effects (font (size 1.27 1.27)) (justify left))
     )
-    (property "Footprint" "Capacitor_SMD:C_0603_1608Metric" (at 192.7098 40.64 0)
+    (property "Footprint" "Capacitor_SMD:C_0402_1005Metric" (at 192.7098 40.64 0)
       (effects (font (size 1.27 1.27)) hide)
     )
@@
       (effects (font (size 1.27 1.27)) (justify left))
     )
-    (property "Footprint" "Capacitor_SMD:C_0603_1608Metric" (at 204.1398 40.64 0)
-      (effects (font (size 1.27 1.27)) hide)
-    )
+    (property "Footprint" "Capacitor_SMD:C_0402_1005Metric" (at 204.1398 40.64 0)
+      (effects (font (size 1.27 1.27)) hide)
+    )
